Commit message: current working version

File: ur5e_egp50_description/urdf/egp50.urdf.xacro (robot description, xacro)
@@ -92,5 +92,5 @@
     <joint name="egp50_tip_joint" type="fixed">
         <parent link="egp50_pincer_link"/>
-	<child link="egp_50_tip" />
+	      <child link="egp_50_tip" />
         <origin xyz="0.0 0.0 ${pincer_height/2}" rpy="0.0 0.0 0.0" />
     </joint>

Commit message: repalce ur_manipulation

File: ur5e_egp50_description/urdf/egp50.urdf.xacro (robot description, xacro)
@@ -39,5 +39,4 @@
       <visual>
         <geometry>
- 	        <!-- <mesh filename="$(find ur_manipulation)/meshes/EGP50.stl" /> -->
           <box size="${body_length} ${body_width} ${body_height}" />
         </geometry>
@@ -47,5 +46,4 @@
       <collision>
         <geometry>
-          <!-- <mesh filename="$(find ur_manipulation)/meshes/EGP50.stl" /> -->
           <box size="${body_length} ${body_width} ${body_height}" />
         </geometry>
